Commit message: EDIT: far planner real version

File: src/mecanum_pkg/mecanum_robot_description/urdf/mecanum_robot_velodyne/mecanum.gazebo.xacro (robot description, xacro)
@@ -59,8 +59,8 @@
     </gazebo> -->
     <gazebo reference="imu_link">
-      <gravity>true</gravity>
+      <gravity>false</gravity>
       <sensor name="imu_sensor" type="imu">
         <always_on>true</always_on>
-        <update_rate>100</update_rate>
+        <update_rate>400</update_rate>
         <visualize>true</visualize>
         <topic>__default_topic__</topic>
@@ -118,4 +118,42 @@
       </sensor>
     </gazebo>
+    <gazebo reference="camera">
+          <sensor name="mecanum_camera_ir" type="depth">
+            <update_rate>0</update_rate>
+            <camera>
+              <horizontal_fov>1.3439</horizontal_fov>
+              <image>
+                <width>640</width>
+                <height>480</height>
+                <format>R8G8B8</format>
+              </image>
+              <clip>
+                <near>0.03</near>
+                <far>100</far>
+              </clip>
+            </camera>
+            <plugin name="mecanum_camera_ir_controller" filename="libgazebo_ros_openni_kinect.so">
+              <baseline>0.2</baseline>
+              <alwaysOn>true</alwaysOn>
+              <update_rate>30</update_rate>
+              <cameraName>camera</cameraName>
+              <imageTopicName>image</imageTopicName>
+              <cameraInfoTopicName>camera_info</cameraInfoTopicName>
+              <depthImageTopicName>depth/image_raw</depthImageTopicName>
+              <depthImageInfoTopicName>depth/camera_info</depthImageInfoTopicName>
+              <pointCloudTopicName>depth/points</pointCloudTopicName>
+              <frameName>camera</frameName>
+              <pointCloudCutoff>0.1</pointCloudCutoff>
+              <pointCloudCutoffMax>15.0</pointCloudCutoffMax>
+              <distortionK1>0.00000001</distortionK1>
+              <distortionK2>0.00000001</distortionK2>
+              <distortionK3>0.00000001</distortionK3>
+              <distortionT1>0.00000001</distortionT1>
+              <distortionT2>0.00000001</distortionT2>
+              <CxPrime>0</CxPrime>
+              <hackBaseline>0</hackBaseline>
+            </plugin>
+          </sensor>
+        </gazebo>
   </xacro:macro>
 </robot>

File: src/mecanum_pkg/mecanum_robot_description/urdf/mecanum_robot_velodyne/mecanum_frame.urdf.xacro (robot description, xacro)
@@ -73,4 +73,5 @@
         <geometry>
           <mesh filename="package://velodyne_description/meshes/VLP16_base_1.dae" />
+          <!-- <box size="0.10 0.10 0.10"/> -->
         </geometry>
       </visual>
@@ -78,4 +79,5 @@
         <geometry>
           <mesh filename="package://velodyne_description/meshes/VLP16_base_2.dae" />
+          <!-- <box size="0.10 0.10 0.10"/> -->
         </geometry>
       </visual>
@@ -102,7 +104,27 @@
         <geometry>
           <mesh filename="package://velodyne_description/meshes/VLP16_scan.dae" />
+              <!-- <box size="0.10 0.10 0.10"/> -->
         </geometry>
       </visual>
     </link>
+      <joint name="camera_joint" type="fixed">
+          <parent link="base_link"/>
+          <child link="camera"/>
+          <origin xyz="0.25 -0.08 0" rpy="0 0 0"/>
+      </joint>
+      <link name="camera">
+          <visual>
+            <origin xyz="0 0 0" rpy="1.57 0 1.57"/>
+            <geometry>
+              <box size="0.05 0.05 0.05"/>
+            </geometry>
+          </visual>
+          <collision>
+            <origin xyz="0.003 0.065 0.007" rpy="0 0 0"/>
+            <geometry>
+              <box size="0.012 0.132 0.020"/>
+            </geometry>
+          </collision>
+      </link>
     </xacro:macro>
 </robot>
